File: sch_pcb/usb_kb.kicad_pcb (KiCad board)
At the start: 0 parts

Commit message: ошибка R11. Конечный вариант
Parts:
- added D1: D_Schottky, Diode_SMD:D_SMA, F.Cu at (123.5, 55.1)
- added D2: LED_ALT, Diode_SMD:D_0805_2012Metric_Pad1.15x1.40mm_HandSolder, F.Cu at (76.9, 81.2)
- added D3: LED_ALT, Diode_SMD:D_0805_2012Metric_Pad1.15x1.40mm_HandSolder, F.Cu at (81.6, 81.2)
- added D4: LED_ALT, Diode_SMD:D_0805_2012Metric_Pad1.15x1.40mm_HandSolder, F.Cu at (121.9, 58.9)
- added J1: Conn_01x04_Female, Connector_PinHeader_2.54mm:PinHeader_1x04_P2.54mm_Vertical, F.Cu at (117.2, 55.2)
- added JP1: Jumper, Jumper:SolderJumper-2_P1.3mm_Open_TrianglePad1.0x1.5mm, F.Cu at (121.7, 62.2)
- added JP2: Jumper, Jumper:SolderJumper-2_P1.3mm_Open_TrianglePad1.0x1.5mm, F.Cu at (126.4, 59.2)
- added P1: USB_C_Plug, Connector_USB:USB_C_Receptacle_HRO_TYPE-C-31-M-12, F.Cu at (93.4, 78.8)
- added SW1: SW_Push, Button_Switch_Keyboard:SW_Cherry_MX_1.00u_PCB, F.Cu at (87.1, 57.9)
- added SW2: SW_Push, Button_Switch_Keyboard:SW_Cherry_MX_1.00u_PCB, F.Cu at (107.3, 57.9)
- added U1: STM32F103C6Tx, Package_QFP:LQFP-48_7x7mm_P0.5mm, F.Cu at (120.5, 70.8)
- added U2: USBLC6-2SC6, Package_TO_SOT_SMD:SOT-23-6, F.Cu at (111.5, 78.8)
- added U3: AMS1117-3.3, Package_TO_SOT_SMD:SOT-223-3_TabPin2, F.Cu at (104.2, 77.2)
- added X1: 8MHz, Crystal:Crystal_HC49-4H_Vertical, F.Cu at (78.6, 76.4)
Other:
- copper layers 0 -> 2
- net class Default added: clearance 0.2, trace_width 0.25, via_dia 0.8, via_drill 0.4
