File: sch_pcb/usb_kb.kicad_pcb (KiCad board)
At the start: 2 copper layers, 14 parts, among them J1 Conn_01x04_Female, P1 USB_C_Plug, SW1 SW_Push, SW2 SW_Push, U1 STM32F103C6Tx, U2 USBLC6-2SC6, U3 AMS1117-3.3, X1 8MHz

Commit message: Новые посадочные места
Parts:
- added C1: 1uF, Capacitor_SMD:C_0805_2012Metric_Pad1.18x1.45mm_HandSolder, F.Cu at (1.91, 1.01)
- added C10: 20pF, Capacitor_SMD:C_0805_2012Metric_Pad1.18x1.45mm_HandSolder, F.Cu at (1.91, 13.0)
- added C11: 100nF, Capacitor_SMD:C_0805_2012Metric_Pad1.18x1.45mm_HandSolder, F.Cu at (16.3, 1.01)
- added C12: 47nF, Capacitor_SMD:C_0805_2012Metric_Pad1.18x1.45mm_HandSolder, F.Cu at (6.72, 10.0)
- added C13: 47nF, Capacitor_SMD:C_0805_2012Metric_Pad1.18x1.45mm_HandSolder, F.Cu at (11.5, 7.03)
- added C14: 0.1uF, Capacitor_SMD:C_0805_2012Metric_Pad1.18x1.45mm_HandSolder, F.Cu at (16.3, 4.02)
- added C15: 0.1uF, Capacitor_SMD:C_0805_2012Metric_Pad1.18x1.45mm_HandSolder, F.Cu at (6.72, 13.0)
- added C2: 0.1uF, Capacitor_SMD:C_0805_2012Metric_Pad1.18x1.45mm_HandSolder, F.Cu at (1.91, 4.02)
- added C3: 1uF, Capacitor_SMD:C_0805_2012Metric_Pad1.18x1.45mm_HandSolder, F.Cu at (6.72, 1.01)
- added C4: 0.1uF, Capacitor_SMD:C_0805_2012Metric_Pad1.18x1.45mm_HandSolder, F.Cu at (1.91, 7.03)
- added C5: 100nF, Capacitor_SMD:C_0805_2012Metric_Pad1.18x1.45mm_HandSolder, F.Cu at (6.72, 4.02)
- added C6: 100nF, Capacitor_SMD:C_0805_2012Metric_Pad1.18x1.45mm_HandSolder, F.Cu at (11.5, 1.01)
- added C7: 100nF, Capacitor_SMD:C_0805_2012Metric_Pad1.18x1.45mm_HandSolder, F.Cu at (1.91, 10.0)
- added C8: 100nF, Capacitor_SMD:C_0805_2012Metric_Pad1.18x1.45mm_HandSolder, F.Cu at (6.72, 7.03)
- added C9: 20pF, Capacitor_SMD:C_0805_2012Metric_Pad1.18x1.45mm_HandSolder, F.Cu at (11.5, 4.02)
- added R1: 20R, Resistor_SMD:R_0805_2012Metric_Pad1.20x1.40mm_HandSolder, F.Cu at (21.1, 0.98)
- added R10: 100, Resistor_SMD:R_0805_2012Metric_Pad1.20x1.40mm_HandSolder, F.Cu at (16.2, 12.9)
- added R11: 10k, Resistor_SMD:R_0805_2012Metric_Pad1.20x1.40mm_HandSolder, F.Cu at (21.1, 9.95)
- added R12: 100, Resistor_SMD:R_0805_2012Metric_Pad1.20x1.40mm_HandSolder, F.Cu at (25.8, 6.88)
- added R13: 10k, Resistor_SMD:R_0805_2012Metric_Pad1.20x1.40mm_HandSolder, F.Cu at (21.0, 12.9)
- added R14: 10k, Resistor_SMD:R_0805_2012Metric_Pad1.20x1.40mm_HandSolder, F.Cu at (25.8, 9.83)
- added R15: 10k, Resistor_SMD:R_0805_2012Metric_Pad1.20x1.40mm_HandSolder, F.Cu at (25.7, 12.9)
- added R2: R, Resistor_SMD:R_0805_2012Metric_Pad1.20x1.40mm_HandSolder, F.Cu at (11.5, 10.0)
- added R3: 10k, Resistor_SMD:R_0805_2012Metric_Pad1.20x1.40mm_HandSolder, F.Cu at (16.3, 7.00)
- added R4: 1M, Resistor_SMD:R_0805_2012Metric_Pad1.20x1.40mm_HandSolder, F.Cu at (21.1, 3.93)
- added R5: 1.5k, Resistor_SMD:R_0805_2012Metric_Pad1.20x1.40mm_HandSolder, F.Cu at (11.5, 13.0)
- added R6: 10k, Resistor_SMD:R_0805_2012Metric_Pad1.20x1.40mm_HandSolder, F.Cu at (25.9, 0.98)
- added R7: 510, Resistor_SMD:R_0805_2012Metric_Pad1.20x1.40mm_HandSolder, F.Cu at (16.3, 9.95)
- added R8: 510, Resistor_SMD:R_0805_2012Metric_Pad1.20x1.40mm_HandSolder, F.Cu at (21.1, 7.00)
- added R9: 510, Resistor_SMD:R_0805_2012Metric_Pad1.20x1.40mm_HandSolder, F.Cu at (25.9, 3.93)

Commit message: Разработал схему
Parts:
- removed C6, C7, C8: 100nF, Capacitor_SMD:C_0805_2012Metric_Pad1.18x1.45mm_HandSolder
- removed D2, D4: LED_ALT, Diode_SMD:D_0805_2012Metric_Pad1.15x1.40mm_HandSolder
- removed R7, R8: 510, Resistor_SMD:R_0805_2012Metric_Pad1.20x1.40mm_HandSolder
- C1, C11, C12, C13, C14, C15, C2, C3, D1, J1, P1, R1, R10, R11, R13, R14, R15, R2, R3, R4, R5, R6, U1, U2, U3, X1: moved to B.Cu
- moved R2 206.2 mm to (204.5, 82.5), turned to 270 degrees
- moved C12 204.7 mm to (201.5, 73.0), turned to 90 degrees
- moved C13 204.0 mm to (204.5, 73.0), turned to 90 degrees
- moved C2 193.3 mm to (183.8, 69.5), turned to 270 degrees
- moved C4 192.5 mm to (184.2, 68.7), turned to 270 degrees
- moved R1 192.4 mm to (198.5, 75.5), turned to 180 degrees
- moved C1 192.2 mm to (181.5, 69.5), turned to 270 degrees
- moved R5 191.7 mm to (190.5, 81.5), turned to 270 degrees
- moved C15 187.2 mm to (182.5, 77.5)
- moved R6 186.4 mm to (191.0, 87.5), turned to 90 degrees
- moved C5 184.3 mm to (179.2, 68.8), turned to 270 degrees
- moved C9 182.5 mm to (174.0, 87.0), turned to 180 degrees
- moved C10 181.8 mm to (168.0, 87.0)
- moved R3 179.8 mm to (182.5, 75.5), turned to 180 degrees
- moved C11 178.5 mm to (178.5, 75.5), turned to 180 degrees
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Routing:
- net GNDD: track 0.00 -> 193.7 mm, vias 0 -> 12
- net +3V3: track 0.00 -> 164.7 mm, vias 0 -> 6
- net /SWDIO: track 0.00 -> 50.2 mm, vias 0 -> 1
- net /SWCLK: track 0.00 -> 46.6 mm, vias 0 -> 3
- net Net-(D1-Pad2): track 0.00 -> 33.7 mm, vias 0 -> 2
- net /USB_D-: track 0.00 -> 27.3 mm
- net /USB_D+: track 0.00 -> 27.2 mm, vias 0 -> 2
- net /Button1: track 0.00 -> 26.8 mm, vias 0 -> 2
- net Net-(C15-Pad1): track 0.00 -> 21.9 mm, vias 0 -> 2
- net Net-(JP1-Pad2): track 0.00 -> 21.5 mm
- net Net-(C10-Pad1): track 0.00 -> 20.2 mm
- net +5V: track 0.00 -> 17.9 mm
- net /RST: track 0.00 -> 15.0 mm
- net Net-(C9-Pad1): track 0.00 -> 14.6 mm
- net Net-(C15-Pad2): track 0.00 -> 13.3 mm, vias 0 -> 1
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- added copper zone on B.Cu, net GNDD
- added copper zone on F.Cu, net GNDD
- added copper zone on B.Cu, net Net-(JP1-Pad2)
- added copper zone on F.Cu, net Net-(JP1-Pad2)
Other:
- board outline added: 46 x 24 mm

Commit message: Переделал схему, добавил дифф пару
Parts:
- C1, C10, C11, C12, C13, C14, C15, C2, C3, C4, C5, C9: footprint Capacitor_SMD:C_0805_2012Metric_Pad1.18x1.45mm_HandSolder -> Capacitor_SMD:C_0603_1608Metric_Pad1.05x0.95mm_HandSolder
- D1: footprint Diode_SMD:D_SMA -> Diode_SMD:D_MiniMELF_Handsoldering
- P1: value USB_C_Plug -> USB_C_Plug_USB2.0
- R1, R10, R11, R12, R13, R14, R15, R2, R3, R4, R5, R6, R9: footprint Resistor_SMD:R_0805_2012Metric_Pad1.20x1.40mm_HandSolder -> Resistor_SMD:R_0603_1608Metric_Pad1.05x0.95mm_HandSolder
- U2: moved to F.Cu
- moved R5 13.4 mm to (200.2, 72.2), turned to 0 degrees
- moved U2 9.38 mm to (200.0, 69.0), turned to 180 degrees
- moved R2 7.92 mm to (200.1, 75.9), turned to 0 degrees
- moved C12 7.01 mm to (204.7, 79.3), turned to 270 degrees
- moved C13 6.76 mm to (201.9, 79.3), turned to 270 degrees
- moved R1 2.02 mm to (200.1, 74.3), turned to 0 degrees
- moved D1 0.86 mm to (200.3, 68.6)
- moved P1 0.07 mm to (197.6, 87.4)
Connections:
- net /USB_D+ renamed /USB_P
- net /USB_D- renamed /USB_N
- net Net-(P1-PadA6) renamed /D_P
- net Net-(P1-PadA7) renamed /D_N
- P1 pad A8: Net-(P1-PadA8) -> (no net)
- P1 pad B8: Net-(P1-PadB8) -> (no net)
Routing:
- net /D_N: track 8.06 -> 21.5 mm
- net /USB_P: track 27.2 -> 39.5 mm
- net /USB_N: track 27.3 -> 39.2 mm, vias 0 -> 1
- net /D_P: track 10.1 -> 18.8 mm
- net GNDD: track 193.7 -> 197.4 mm
- net +3V3: track 164.7 -> 160.9 mm, vias 6 -> 5
- net Net-(D1-Pad2): track 33.7 -> 30.7 mm
- net /SWDIO: track 50.2 -> 51.2 mm
- net Net-(JP2-Pad1): track 6.81 -> 7.80 mm
- net +5V: track 17.9 -> 18.4 mm
Other:
- rule via_min_size: 0.4 -> 0.2
- board text added: "github.com/TakitaNirasa/usb_kb"

Commit message: Добавил герберы
Other:
- board text added: "MVP"
Changed lines of the file:
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@@
   (general
     (thickness 1.6)
-    (drawings 5)
+    (drawings 7)
     (tracks 431)
     (zones 0)
@@
   (page A4)
   (layers
-    (0 F.Cu signal hide)
+    (0 F.Cu signal)
     (31 B.Cu signal)
-    (32 B.Adhes user hide)
-    (33 F.Adhes user hide)
-    (34 B.Paste user hide)
+    (32 B.Adhes user)
+    (33 F.Adhes user)
+    (34 B.Paste user)
     (35 F.Paste user hide)
-    (36 B.SilkS user hide)
+    (36 B.SilkS user)
     (37 F.SilkS user)
     (38 B.Mask user hide)
-    (39 F.Mask user)
+    (39 F.Mask user hide)
     (40 Dwgs.User user hide)
     (41 Cmts.User user hide)
@@
     (user_trace_width 0.2)
     (trace_clearance 0.2)
-    (zone_clearance 0.2)
+    (zone_clearance 0.254)
     (zone_45_only no)
     (trace_min 0.2)
@@
     (pcbplotparams
       (layerselection 0x010fc_ffffffff)
-      (usegerberextensions false)
-      (usegerberattributes true)
-      (usegerberadvancedattributes true)
-      (creategerberjobfile true)
+      (usegerberextensions true)
+      (usegerberattributes false)
+      (usegerberadvancedattributes false)
+      (creategerberjobfile false)
       (excludeedgelayer true)
       (linewidth 0.100000)
@@
       (psa4output false)
       (plotreference true)
-      (plotvalue true)
+      (plotvalue false)
       (plotinvisibletext false)
       (padsonsilk false)
-      (subtractmaskfromsilk false)
+      (subtractmaskfromsilk true)
       (outputformat 1)
       (mirror false)
-      (drillshape 1)
+      (drillshape 0)
       (scaleselection 1)
       (outputdirectory ""))
@@
     (tags "usb usb-c 2.0 pd")
     (attr smd)
-    (fp_text reference P1 (at 0 5.645 180) (layer B.SilkS)
-      (effects (font (size 1 1) (thickness 0.15)) (justify mirror))
-    )
-    (fp_text value USB_C_Plug_USB2.0 (at 0 -5.1 180) (layer B.Fab)
-      (effects (font (size 1 1) (thickness 0.15)) (justify mirror))
-    )
-    (fp_line (start -4.7 -3.9) (end 4.7 -3.9) (layer B.SilkS) (width 0.12))
+    (fp_text reference P1 (at 0 5.645) (layer B.SilkS)
+      (effects (font (size 1 1) (thickness 0.15)) (justify mirror))
+    )
+    (fp_text value USB_C_Plug_USB2.0 (at 0 -5.1) (layer B.Fab)
+      (effects (font (size 1 1) (thickness 0.15)) (justify mirror))
+    )
     (fp_line (start -4.47 3.65) (end 4.47 3.65) (layer B.Fab) (width 0.1))
     (fp_line (start -4.47 3.65) (end -4.47 -3.65) (layer B.Fab) (width 0.1))
     (fp_line (start -4.47 -3.65) (end 4.47 -3.65) (layer B.Fab) (width 0.1))
     (fp_line (start 4.47 3.65) (end 4.47 -3.65) (layer B.Fab) (width 0.1))
-    (fp_text user %R (at 0 0 180) (layer B.Fab)
-      (effects (font (size 1 1) (thickness 0.15)) (justify mirror))
-    )
+    (fp_text user %R (at 0 0) (layer B.Fab)
+      (effects (font (size 1 1) (thickness 0.15)) (justify mirror))
+    )
+    (fp_line (start -5.32 5.27) (end 5.32 5.27) (layer B.CrtYd) (width 0.05))
+    (fp_line (start -5.32 -4.15) (end 5.32 -4.15) (layer B.CrtYd) (width 0.05))
+    (fp_line (start -5.32 5.27) (end -5.32 -4.15) (layer B.CrtYd) (width 0.05))
+    (fp_line (start 5.32 5.27) (end 5.32 -4.15) (layer B.CrtYd) (width 0.05))
     (fp_line (start 4.7 1.9) (end 4.7 -0.1) (layer B.SilkS) (width 0.12))
-    (fp_line (start 4.7 -2) (end 4.7 -3.9) (layer B.SilkS) (width 0.12))
     (fp_line (start -4.7 1.9) (end -4.7 -0.1) (layer B.SilkS) (width 0.12))
-    (fp_line (start -4.7 -2) (end -4.7 -3.9) (layer B.SilkS) (width 0.12))
     (pad B1 smd rect (at 3.25 4.045 180) (size 0.6 1.45) (layers B.Cu B.Paste B.Mask)
       (net 5 GNDD))
@@
     )
   )
+  (gr_text "MVP\n" (at 165 70) (layer F.SilkS)
+    (effects (font (size 1 1) (thickness 0.15)))
+  )
+  (gr_poly (pts (xy 162.8 67.2) (xy 163 67.2) (xy 163 67.6) (xy 164.4 67.6) (xy 164.4 67.8) (xy 164.6 67.8) (xy 164.6 68) (xy 166 68) (xy 166 68.2) (xy 165.2 68.2) (xy 165.2 68.4) (xy 165.8 68.4) (xy 165.8 68.6) (xy 165 68.6) (xy 165 68.8) (xy 163.6 68.8) (xy 163.6 69) (xy 163.4 69) (xy 163.4 69.2) (xy 163.2 69.2) (xy 163.2 69.6) (xy 163 69.6) (xy 163 69.8) (xy 162.8 69.8) (xy 162.8 68.2) (xy 162.6 68.2) (xy 162.6 68) (xy 162.4 68) (xy 162.4 67.8) (xy 161.6 67.8) (xy 161.6 67.6) (xy 161.8 67.6) (xy 161.8 67.4) (xy 162 67.4) (xy 162 67.2) (xy 162.2 67.2) (xy 162.2 67) (xy 162.4 67) (xy 162.4 66.8) (xy 162.8 66.8)) (layer F.SilkS) (width 0.01))
   (gr_text github.com/TakitaNirasa/usb_kb (at 173.725 89.025) (layer F.SilkS)
     (effects (font (size 1 1) (thickness 0.15)))
@@
   (segment (start 160.674998 78.754998) (end 160.674998 74.525002) (width 0.25) (layer B.Cu) (net 5))
   (via (at 172.55 69.225) (size 0.8) (drill 0.4) (layers F.Cu B.Cu) (net 5))
-  (segment (start 163.175001 78.715001) (end 163.175001 86.675001) (width 0.25) (layer F.Cu) (net 6))
-  (segment (start 162 77.54) (end 163.175001 78.715001) (width 0.25) (layer F.Cu) (net 6))
-  (via (at 165.5 89) (size 0.8) (drill 0.4) (layers F.Cu B.Cu) (net 6))
-  (segment (start 163.175001 86.675001) (end 165.5 89) (width 0.25) (layer F.Cu) (net 6))
-  (segment (start 165.899999 89.399999) (end 175.600001 89.399999) (width 0.25) (layer B.Cu) (net 6))
-  (segment (start 165.5 89) (end 165.899999 89.399999) (width 0.25) (layer B.Cu) (net 6))
   (via (at 177 88.5) (size 0.8) (drill 0.4) (layers F.Cu B.Cu) (net 6))
-  (segment (start 176.5 88.5) (end 177 88.5) (width 0.25) (layer B.Cu) (net 6))
-  (segment (start 175.600001 89.399999) (end 176.5 88.5) (width 0.25) (layer B.Cu) (net 6))
   (segment (start 177 88.5) (end 187 88.5) (width 0.25) (layer F.Cu) (net 6))
   (via (at 187.5 88) (size 0.8) (drill 0.4) (layers F.Cu B.Cu) (net 6))
@@
   (segment (start 168.5 72.6) (end 163.56 77.54) (width 0.25) (layer B.Cu) (net 6))
   (segment (start 168.5 72) (end 168.5 72.6) (width 0.25) (layer B.Cu) (net 6))
+  (segment (start 176.5 88.5) (end 177 88.5) (width 0.25) (layer B.Cu) (net 6))
+  (segment (start 165.899999 89.399999) (end 175.600001 89.399999) (width 0.25) (layer B.Cu) (net 6))
+  (segment (start 164.425 87.925) (end 165.899999 89.399999) (width 0.25) (layer B.Cu) (net 6))
+  (segment (start 175.600001 89.399999) (end 176.5 88.5) (width 0.25) (layer B.Cu) (net 6))
+  (segment (start 163.175001 78.715001) (end 162 77.54) (width 0.25) (layer F.Cu) (net 6))
+  (segment (start 163.175001 86.675001) (end 163.175001 78.715001) (width 0.25) (layer F.Cu) (net 6))
+  (segment (start 164.425 87.925) (end 163.175001 86.675001) (width 0.25) (layer F.Cu) (net 6))
+  (via (at 164.425 87.925) (size 0.8) (drill 0.4) (layers F.Cu B.Cu) (net 6))
   (segment (start 164.5 86.16319) (end 164.5 77.5) (width 0.25) (layer F.Cu) (net 7))
   (segment (start 164.5 77.5) (end 162 75) (width 0.25) (layer F.Cu) (net 7))
@@
   (segment (start 191 89.1) (end 191 88.375) (width 0.2) (layer B.Cu) (net 16))
   (segment (start 190.82501 89.27499) (end 191 89.1) (width 0.2) (layer B.Cu) (net 16))
-  (segment (start 187.1625 85.25) (end 188.176998 85.25) (width 0.25) (layer B.Cu) (net 47))
   (segment (start 178.084278 83.75) (end 178.8375 83.75) (width 0.25) (layer B.Cu) (net 39))
   (segment (start 178.059288 83.77499) (end 178.084278 83.75) (width 0.25) (layer B.Cu) (net 39))
@@
   (segment (start 183.75 77.75) (end 183.5 77.5) (width 0.25) (layer B.Cu) (net 46))
   (segment (start 185 77.75) (end 183.75 77.75) (width 0.25) (layer B.Cu) (net 46))
+  (segment (start 187.1625 85.25) (end 188.176998 85.25) (width 0.25) (layer B.Cu) (net 47))
   (segment (start 199.25 75.9) (end 198.286397 75.9) (width 0.2) (layer B.Cu) (net 47))
   (segment (start 188.238998 85.225) (end 187.1875 85.225) (width 0.2) (layer B.Cu) (net 47))
